Commit message: urdf and readme updates

File: ROS/src/dogbot_description/urdf/dogbot.urdf (robot description, URDF)
Before this commit: robot dogbot, 18 links, 17 joints
Links:
- added link bodytext, mass 0.001; visual mesh filename=package://dogbot_description/meshes/bodyTEXT.dae scale=1.0 1.0 1.0
- link back_left_foot: geometry collision sphere radius=0.028; visual mesh filename=package://dogbot_description/meshes/foot.dae scale=1.0 1.0 1.0
- link back_left_hip: geometry collision cylinder length=0.08 radius=0.0525; visual mesh filename=package://dogbot_description/meshes/hip.dae scale=1.0 1.0 1.0
- link back_left_lowerleg: geometry collision box size=0.02 0.017 0.065; collision box size=0.02 0.017 0.065
- link back_left_upperleg: geometry collision box size=0.025 0.084 0.27; collision box size=0.026 0.074 0.138
- link back_right_foot: geometry collision sphere radius=0.028; visual mesh filename=package://dogbot_description/meshes/foot.dae scale=1.0 1.0 1.0
- link back_right_hip: geometry collision cylinder length=0.08 radius=0.0525; visual mesh filename=package://dogbot_description/meshes/hip.dae scale=1.0 1.0 1.0
- link back_right_lowerleg: geometry collision box size=0.02 0.017 0.065; collision box size=0.02 0.017 0.065
- link back_right_upperleg: geometry collision box size=0.025 0.084 0.27; collision box size=0.026 0.074 0.138
- link body: geometry collision box size=0.035 0.132 0.105; collision box size=0.035 0.132 0.105
- link front_left_foot: geometry collision sphere radius=0.028; visual mesh filename=package://dogbot_description/meshes/foot.dae scale=1.0 1.0 1.0
- link front_left_hip: geometry collision cylinder length=0.08 radius=0.0525; visual mesh filename=package://dogbot_description/meshes/hip.dae scale=1.0 1.0 1.0
- link front_left_lowerleg: geometry collision box size=0.02 0.017 0.065; collision box size=0.02 0.017 0.065
- link front_left_upperleg: geometry collision box size=0.025 0.084 0.27; collision box size=0.026 0.074 0.138
- link front_right_foot: geometry collision sphere radius=0.028; visual mesh filename=package://dogbot_description/meshes/foot.dae scale=1.0 1.0 1.0
- link front_right_hip: geometry collision cylinder length=0.08 radius=0.0525; visual mesh filename=package://dogbot_description/meshes/hip.dae scale=1.0 1.0 1.0
- link front_right_lowerleg: geometry collision box size=0.02 0.017 0.065; collision box size=0.02 0.017 0.065
- link front_right_upperleg: geometry collision box size=0.025 0.084 0.27; collision box size=0.026 0.074 0.138
Joints:
- added joint bodytext_joint: type fixed, parent body, child bodytext
- joint back_left_pitch_joint: limit lower=-6.28318530718 upper=6.28318530718 effort=1000 velocity=6.0 -> lower=-1.57079632679 upper=3.14159265359 effort=1000 velocity=6.0
- joint back_right_pitch_joint: limit lower=-6.28318530718 upper=6.28318530718 effort=1000 velocity=6.0 -> lower=-3.14159265359 upper=1.57079632679 effort=1000 velocity=6.0
- joint front_left_pitch_joint: limit lower=-6.28318530718 upper=6.28318530718 effort=1000 velocity=6.0 -> lower=-1.57079632679 upper=3.14159265359 effort=1000 velocity=6.0
- joint front_right_pitch_joint: limit lower=-6.28318530718 upper=6.28318530718 effort=1000 velocity=6.0 -> lower=-3.14159265359 upper=1.57079632679 effort=1000 velocity=6.0

File: ROS/src/dogbot_description/urdf/dogbot.xacro (robot description, xacro)
@@ -1,4 +1,8 @@
 <?xml version="1.0"?>
 <robot name="dogbot" xmlns:xacro="http://ros.org/wiki/xacro">
+<!-- =================================================================================== -->
+<!-- |    Details of mass and inertia in this file are estimates only                  | -->
+<!-- |    as DogBot design is still undergoing refinements                             | -->
+<!-- =================================================================================== -->
   <xacro:property name="collisionmesh" value="false" />
   <xacro:property name="bodyheight" value="0.105" />
@@ -12,5 +16,6 @@
   <xacro:property name="kp" value="1000000" />
   <xacro:property name="kd" value="1.0" />
-  <xacro:property name="d2rad" value="0.017453" /><!-- degrees to radians -->
+  <!-- degrees to radians -->
+  <xacro:property name="d2rad" value="0.017453" />
   <material name="blue">
     <color rgba="0 0 0.8 1"/>
@@ -22,13 +27,16 @@
     <color rgba="1 1 1 1"/>
   </material>
+  <material name="dogbotred">
+    <color rgba="1 0 0 1"/>
+  </material>
   <material name="dogbotgray">
     <color rgba="0.7 0.7 0.7 1"/>
   </material>
+  <!-- Approximate mass distribution with a box
+  set ifactor=1 for solid box, =2.0 for a thin shell -->
   <xacro:macro name="default_inertial" params="mass xSize ySize zSize x:=0 y:=0 z:=0 ifactor:=1.0">
     <inertial>
       <mass value="${mass}" />
       <origin xyz="${x} ${y} ${z}" rpy="0 0 0" />
-      <!-- Approximate mass distribution with a box
-      set ifactor=1 for solid box, =2.0 for a thin shell -->
       <inertia
         ixx="${(1.0 / 12.0) * mass * ifactor * (pow(ySize, 2) + pow(zSize, 2))}"
@@ -41,4 +49,8 @@
     </inertial>
   </xacro:macro>
+  <!-- useful for visual-only links; need some inertia on all elements -->
+  <xacro:macro name="tinymass" >
+    <xacro:default_inertial mass="0.001" xSize="0.001" ySize="0.001" zSize="0.001" />
+  </xacro:macro>
   <xacro:macro name="custom_inertial" params="mass x:=0 y:=0 z:=0 r:=0 p:=0 yaw:=0 ixx:=0.01 ixy:=0 ixz:=0 iyy:=0.01 iyz:=0 izz:=0.01">
     <inertial>
@@ -76,13 +88,13 @@
   <link name="body">
     <visual>
-      <geometry>
-        <mesh scale="0.001 0.001 0.001" filename="package://dogbot_description/meshes/body.stl"/>
-      </geometry>
-      <material name="white"/>
+      <origin xyz="0 0 0" rpy="${-0.5 * pi} 0 0" />
+      <geometry>
+        <mesh scale="1.0 1.0 1.0" filename="package://dogbot_description/meshes/body.dae"/>
+      </geometry>
     </visual>
     <xacro:if value="${collisionmesh}">
     <collision>
       <geometry>
-        <mesh scale="0.001 0.001 0.001" filename="package://dogbot_description/meshes/body.stl"/>
+        <mesh scale="1.0 1.0 1.0" filename="package://dogbot_description/meshes/body.dae"/>
       </geometry>
     </collision>
@@ -108,4 +120,17 @@
     <child link="body"/>
   </joint>
+  <link name="bodytext">
+    <visual>
+      <origin xyz="0 0 0" rpy="${-0.5 * pi} 0 0" />
+      <geometry>
+        <mesh scale="1.0 1.0 1.0" filename="package://dogbot_description/meshes/bodyTEXT.dae"/>
+      </geometry>
+    </visual>
+    <xacro:tinymass />
+  </link>
+  <joint name="bodytext_joint" type="fixed">
+    <parent link="body"/>
+    <child link="bodytext"/>
+  </joint>
   <gazebo reference="body">
     <mu1 value="200.0"/>
@@ -113,5 +138,4 @@
     <kp value="${kp}" />
     <kd value="${kd}" />
-    <material>Gazebo/white</material>
   </gazebo>
   <!-- reflectx indicates left/right, reflecty indicates front/back (front-right is 1,1, i.e.
@@ -121,15 +145,14 @@
     <link name="${prefix}_${suffix}_hip">
       <visual>
-        <origin xyz="0 0 0" rpy="0 ${(reflectx-1) * 0.5 * pi} 0" />
-        <geometry>
-          <mesh scale="0.001 0.001 0.001" filename="package://dogbot_description/meshes/hip.stl"/>
-        </geometry>
-        <material name="white"/>
+        <origin xyz="0 0 0" rpy="${-0.5 * pi} ${(reflectx-1) * 0.5 * pi} 0" />
+        <geometry>
+          <mesh scale="1.0 1.0 1.0" filename="package://dogbot_description/meshes/hip.dae"/>
+        </geometry>
       </visual>
       <xacro:if value="${collisionmesh}">
       <collision>
-        <origin xyz="0 0 0" rpy="0 ${(reflectx-1) * 0.5 * pi} 0" />
-        <geometry>
-          <mesh scale="0.001 0.001 0.001" filename="package://dogbot_description/meshes/hip.stl"/>
+        <origin xyz="0 0 0" rpy="${-0.5 * pi} ${(reflectx-1) * 0.5 * pi} 0" />
+        <geometry>
+          <mesh scale="1.0 1.0 1.0" filename="package://dogbot_description/meshes/hip.dae"/>
         </geometry>
       </collision>
@@ -145,5 +168,5 @@
       <parent link="body"/>
       <child link="${prefix}_${suffix}_hip"/>
-      <origin xyz="${hipoffsetside*reflectx} ${hipoffset * reflecty} 0" rpy="0 0 0"/><!-- "0 0 ${-pi*(1-reflecty)/2}"/> -->
+      <origin xyz="${hipoffsetside*reflectx} ${hipoffset * reflecty} 0" rpy="0 0 0"/>
       <limit
          lower ="${-100 * d2rad}"
@@ -153,15 +176,14 @@
     <link name="${prefix}_${suffix}_upperleg">
       <visual>
-        <origin xyz="0 0 0" rpy="0 0 ${ (reflectx -1) * 0.5 * pi}" />
-        <geometry>
-          <mesh scale="0.001 0.001 0.001" filename="package://dogbot_description/meshes/leg_upper.stl"/>
-        </geometry>
-        <material name="white"/>
+        <origin xyz="0 0 0" rpy="${-0.5 * pi} 0 ${ (reflectx -1) * 0.5 * pi}" />
+        <geometry>
+          <mesh scale="1.0 1.0 1.0" filename="package://dogbot_description/meshes/LegUpper_withCover.dae"/>
+        </geometry>
       </visual>
       <xacro:if value="${collisionmesh}">
       <collision>
-        <origin xyz="0 0 0" rpy="0 0 ${ (reflectx -1) * 0.5 * pi}" />
-        <geometry>
-          <mesh scale="0.001 0.001 0.001" filename="package://dogbot_description/meshes/leg_upper.stl"/>
+        <origin xyz="0 0 0" rpy="${-0.5 * pi} 0 ${ (reflectx -1) * 0.5 * pi}" />
+        <geometry>
+          <mesh scale="1.0 1.0 1.0" filename="package://dogbot_description/meshes/LegUpper_withCover.dae"/>
         </geometry>
       </collision>
@@ -188,6 +210,6 @@
       <origin xyz="${(legoffsetside - hipoffsetside)*reflectx} 0 0" rpy="0 0 0"/>
       <limit
-        lower ="-${pi*2}"
-        upper="${pi*2}"
+        lower ="${-0.5 * pi *(reflectx+1) + 0.25 * pi * (reflectx-1)}"
+        upper="${0.25 * pi *(reflectx+1) - 0.5 * pi * (reflectx-1)}"
         effort="1000"
         velocity="6.0"
@@ -196,15 +218,14 @@
     <link name="${prefix}_${suffix}_lowerleg">
       <visual>
-        <origin xyz="0 0 0" rpy="0 0 0" />
-        <geometry>
-          <mesh scale="0.001 0.001 0.001" filename="package://dogbot_description/meshes/leg_lower_CF.stl"/>
-        </geometry>
-        <material name="white"/>
+        <origin xyz="0 0 0" rpy="${-0.5 * pi} 0 0" />
+        <geometry>
+          <mesh scale="1.0 1.0 1.0" filename="package://dogbot_description/meshes/LegLower_nofoot.dae"/>
+        </geometry>
       </visual>
       <xacro:if value="${collisionmesh}">
       <collision>
-        <origin xyz="0 0 0" rpy="0 0 0" />
-        <geometry>
-          <mesh scale="0.001 0.001 0.001" filename="package://dogbot_description/meshes/leg_lower_CF.stl"/>
+        <origin xyz="0 0 0" rpy="${-0.5 * pi} 0 0" />
+        <geometry>
+          <mesh scale="1.0 1.0 1.0" filename="package://dogbot_description/meshes/LegLower_nofoot.dae"/>
         </geometry>
       </collision>
@@ -227,5 +248,4 @@
       <kd value="${kd}" />
       <selfCollide value="true" />
-      <material>Gazebo/Grey</material>
     </gazebo>
     <joint name="${prefix}_${suffix}_knee_joint" type="revolute">
@@ -242,14 +262,14 @@
     <link name="${prefix}_${suffix}_foot">
       <visual>
-        <origin xyz="0 0 0" rpy="0 0 0" />
-        <geometry>
-          <mesh scale="0.001 0.001 0.001" filename="package://dogbot_description/meshes/leg_lower_FOOT.stl"/>
+        <origin xyz="0 0 0" rpy="${-0.5 * pi} 0 0" />
+        <geometry>
+          <mesh scale="1.0 1.0 1.0" filename="package://dogbot_description/meshes/foot.dae"/>
         </geometry>
       </visual>
       <xacro:if value="${collisionmesh}">
       <collision>
-        <origin xyz="0 0 0" rpy="0 0 0" />
-        <geometry>
-          <mesh scale="0.001 0.001 0.001" filename="package://dogbot_description/meshes/leg_lower_FOOT.stl"/>
+        <origin xyz="0 0 0" rpy="${-0.5 * pi} 0 0" />
+        <geometry>
+          <mesh scale="1.0 1.0 1.0" filename="package://dogbot_description/meshes/foot.dae"/>
         </geometry>
       </collision>
@@ -276,5 +296,4 @@
       <kp value="${kp}" />
       <kd value="${kd}" />
-      <material>Gazebo/Red</material>
     </gazebo>
     <transmission name="${prefix}_${suffix}_roll_transmition" >

Commit message: urdf update joint effort limit

File: ROS/src/dogbot_description/urdf/dogbot.urdf (robot description, URDF)
Before this commit: robot dogbot, 19 links, 18 joints
Links:
- link back_left_foot: mass 0.2 -> 0.001
- link back_left_hip: mass 0.852 -> 0.836
- link back_left_lowerleg: mass 0.45 -> 0.302
- link back_left_upperleg: mass 2.791 -> 1.851
- link back_right_foot: mass 0.2 -> 0.001
- link back_right_hip: mass 0.852 -> 0.836
- link back_right_lowerleg: mass 0.45 -> 0.302
- link back_right_upperleg: mass 2.791 -> 1.851
- link body: mass 9.836 -> 9.3
- link front_left_foot: mass 0.2 -> 0.001
- link front_left_hip: mass 0.852 -> 0.836
- link front_left_lowerleg: mass 0.45 -> 0.302
- link front_left_upperleg: mass 2.791 -> 1.851
- link front_right_foot: mass 0.2 -> 0.001
- link front_right_hip: mass 0.852 -> 0.836
- link front_right_lowerleg: mass 0.45 -> 0.302
- link front_right_upperleg: mass 2.791 -> 1.851
Joints:
- joint back_left_knee_joint: limit lower=-2.61795 upper=0.02 effort=1000 velocity=6.0 -> lower=-2.61795 upper=0.02 effort=60 velocity=6.0
- joint back_left_pitch_joint: limit lower=-1.57079632679 upper=3.14159265359 effort=1000 velocity=6.0 -> lower=-1.57079632679 upper=3.14159265359 effort=60 velocity=6.0
- joint back_left_roll_joint: limit lower=-1.7453 upper=1.7453 effort=500 velocity=6.0 -> lower=-1.7453 upper=1.7453 effort=60 velocity=6.0
- joint back_right_knee_joint: limit lower=-0.02 upper=2.61795 effort=1000 velocity=6.0 -> lower=-0.02 upper=2.61795 effort=60 velocity=6.0
- joint back_right_pitch_joint: limit lower=-3.14159265359 upper=1.57079632679 effort=1000 velocity=6.0 -> lower=-3.14159265359 upper=1.57079632679 effort=60 velocity=6.0
- joint back_right_roll_joint: limit lower=-1.7453 upper=1.7453 effort=500 velocity=6.0 -> lower=-1.7453 upper=1.7453 effort=60 velocity=6.0
- joint front_left_knee_joint: limit lower=-2.61795 upper=0.02 effort=1000 velocity=6.0 -> lower=-2.61795 upper=0.02 effort=60 velocity=6.0
- joint front_left_pitch_joint: limit lower=-1.57079632679 upper=3.14159265359 effort=1000 velocity=6.0 -> lower=-1.57079632679 upper=3.14159265359 effort=60 velocity=6.0
- joint front_left_roll_joint: limit lower=-1.7453 upper=1.7453 effort=500 velocity=6.0 -> lower=-1.7453 upper=1.7453 effort=60 velocity=6.0
- joint front_right_knee_joint: limit lower=-0.02 upper=2.61795 effort=1000 velocity=6.0 -> lower=-0.02 upper=2.61795 effort=60 velocity=6.0
- joint front_right_pitch_joint: limit lower=-3.14159265359 upper=1.57079632679 effort=1000 velocity=6.0 -> lower=-3.14159265359 upper=1.57079632679 effort=60 velocity=6.0
- joint front_right_roll_joint: limit lower=-1.7453 upper=1.7453 effort=500 velocity=6.0 -> lower=-1.7453 upper=1.7453 effort=60 velocity=6.0

File: ROS/src/dogbot_description/urdf/dogbot.xacro (robot description, xacro)
@@ -8,6 +8,8 @@
      |    Author:  Nic Greenway, nic@reactrobotics.com
      |
-     |    Note: details of mass and inertia in this file are estimates only
-     |    as DogBot design is still undergoing refinements                             |
+     |    Note: some details of mass and inertia in this file are estimates,
+     |    as DogBot design is still undergoing refinements, and values will vary
+     |    with individual DogBot specification (e.g. battery configuration, on-board
+     |    processor, etc.)
      =================================================================================== -->
   <xacro:property name="collisionmesh" value="false" />
@@ -119,5 +121,5 @@
       <xacro:offset_cylinderpair l="0.080" y="-0.3975" />
     </xacro:unless>
-    <xacro:default_inertial mass="9.836" xSize="${bodywidth}" ySize="${bodylen}" zSize="${bodyheight}" ifactor="1.5" />
+    <xacro:custom_inertial mass="9.3" ixx="0.41" iyy="0.091" izz="0.482"/>
   </link>
   <joint name="base_joint" type="fixed">
@@ -167,5 +169,5 @@
         <xacro:offset_cylinder l="0.08" p="${pi/2}" x="${0.02 * reflectx}"/>
       </xacro:unless>
-      <xacro:default_inertial mass="0.852" xSize="${bodyheight}" ySize="0.08" zSize="${bodyheight}" z="0.007" ifactor="1.2"/>
+      <xacro:custom_inertial mass="0.836" x="${0.0074 * reflectx}" ixx="0.00213" iyy="0.00147" izz="0.00172"/>
     </link>
     <!-- roll joint connects the hip to the body -->
@@ -178,5 +180,5 @@
          lower ="${-100 * d2rad}"
          upper ="${100 * d2rad}"
-         effort="500" velocity="6.0" />
+         effort="60" velocity="6.0" />
     </joint>
     <link name="${prefix}_${suffix}_upperleg">
@@ -207,5 +209,5 @@
         <xacro:offset_cylinder l="0.013" rad="0.017" z="${-upperleglen}" p="${pi/2}" x="${-0.036 * reflectx}" />
       </xacro:unless>
-      <xacro:default_inertial mass="2.791" xSize="0.08" ySize="0.03" zSize="0.38" ifactor="1.3" x="0.0129" z="-0.0785" />
+      <xacro:custom_inertial mass="1.851" x="${0.0418 * reflectx}" z="-0.0517" ixx="0.0238" iyy="0.0252" izz="0.0044"/>
     </link>
     <!-- pitch joint connects hip to upper leg -->
@@ -218,5 +220,5 @@
         lower ="${-0.5 * pi *(reflectx+1) + 0.25 * pi * (reflectx-1)}"
         upper="${0.25 * pi *(reflectx+1) - 0.5 * pi * (reflectx-1)}"
-        effort="1000"
+        effort="60"
         velocity="6.0"
       />
@@ -246,5 +248,5 @@
         <xacro:offset_cylinder l="0.290" rad="0.006" p="-0.04996" x="-0.01575" y="-0.0375" z="-0.145" />
       </xacro:unless>
-      <xacro:default_inertial mass="0.45" xSize="0.03" ySize="0.02" zSize="0.36" y="-0.02" z="-0.03" ifactor="1.7" />
+      <xacro:custom_inertial mass="0.302" y="-0.029" z="-0.1439" ixx="0.00527" iyy="0.00509" izz="0.0008"/>
     </link>
     <gazebo reference="${prefix}_${suffix}_lowerleg">
@@ -263,5 +265,5 @@
          lower ="${-0.01*(reflectx+1) + 150 * d2rad * (reflectx-1)/2}"
          upper ="${-0.01*(reflectx-1) + 150 * d2rad * (reflectx+1)/2}"
-         effort="1000" velocity="6.0"
+         effort="60" velocity="6.0"
        />
     </joint>
@@ -289,5 +291,6 @@
         </collision>
       </xacro:unless>
-      <xacro:default_inertial mass="0.2" xSize="0.05" ySize="0.05" zSize="0.05" y="-0.035" z="${-lowerleglen}"/>
+      <!-- foot mass is included in lower leg link -->
+      <xacro:tinymass />
     </link>
     <joint name="${prefix}_${suffix}_foot_joint" type="fixed">

Commit message: urdf updated to fix slight error in body length

File: ROS/src/dogbot_description/urdf/dogbot.urdf (robot description, URDF)
Before this commit: robot dogbot, 19 links, 18 joints
Joints:
- joint back_left_knee_joint: axis -1 0 0 -> 1 0 0
- joint back_left_roll_joint: origin xyz=-0.088 -0.2795 0 rpy=0 0 0 -> xyz=-0.088 -0.2875 0 rpy=0 0 0
- joint back_right_knee_joint: axis 1 0 0 -> -1 0 0
- joint back_right_roll_joint: origin xyz=0.088 -0.2795 0 rpy=0 0 0 -> xyz=0.088 -0.2875 0 rpy=0 0 0
- joint front_left_knee_joint: axis -1 0 0 -> 1 0 0
- joint front_left_roll_joint: origin xyz=-0.088 0.2795 0 rpy=0 0 0 -> xyz=-0.088 0.2875 0 rpy=0 0 0
- joint front_right_knee_joint: axis 1 0 0 -> -1 0 0
- joint front_right_roll_joint: origin xyz=0.088 0.2795 0 rpy=0 0 0 -> xyz=0.088 0.2875 0 rpy=0 0 0

File: ROS/src/dogbot_description/urdf/dogbot.xacro (robot description, xacro)
@@ -18,5 +18,5 @@
   <xacro:property name="bodylen" value="0.865" />
   <xacro:property name="hipoffsetside" value="0.088" /><!-- offset from body centreline to hip roll -->
-  <xacro:property name="hipoffset" value="0.2795" /><!-- offset from body midpoint front/back to hip -->
+  <xacro:property name="hipoffset" value="0.2875" /><!-- offset from body midpoint front/back to hip, axis-to-axis is 575mm -->
   <xacro:property name="legoffsetside" value="0.18675" /><!-- from centreline to centre/origin of upper leg -->
   <xacro:property name="upperleglen" value="0.315" />
@@ -258,5 +258,5 @@
     </gazebo>
     <joint name="${prefix}_${suffix}_knee_joint" type="revolute">
-      <axis xyz="${reflectx} 0 0" rpy="${-2*pi} 0 0" />
+      <axis xyz="${-1 * reflectx} 0 0" rpy="${-2*pi} 0 0" />
       <parent link="${prefix}_${suffix}_upperleg"/>
       <child link="${prefix}_${suffix}_lowerleg"/>
